Commit message: feat: add joint damping

File: gazebo_dart_model_pose_bug/stick_description/stick.urdf.xacro (robot description, xacro)
@@ -115,4 +115,5 @@
     <axis xyz="0 0 1"/>
     <limit acceleration="15" lower="-2.9671" effort="87" upper="2.9671" velocity="2.5"/>
+    <dynamics damping="0.003"/>
   </joint>
   <joint name="$(arg robot_name)_joint2" type="revolute">
@@ -122,4 +123,5 @@
     <axis xyz="0 0 1"/>
     <limit acceleration="15" lower="-2.9671" effort="87" upper="2.9671" velocity="2.5"/>
+    <dynamics damping="0.003"/>
   </joint>
   <joint name="$(arg robot_name)_joint3" type="revolute">
@@ -129,4 +131,5 @@
     <axis xyz="0 0 1"/>
     <limit acceleration="15" lower="-2.9671" effort="87" upper="2.9671" velocity="2.5"/>
+    <dynamics damping="0.003"/>
   </joint>
   <joint name="$(arg robot_name)_joint4" type="revolute">
@@ -136,4 +139,5 @@
     <axis xyz="0 0 1"/>
     <limit acceleration="15" lower="-2.9671" effort="87" upper="2.9671" velocity="2.5"/>
+    <dynamics damping="0.003"/>
   </joint>
   <!--Create hardware interfaces-->
